Commit message: updated with visual meshes

File: urdf/irb4600_60_205.urdf (robot description, URDF)
Before this commit: robot abb_irb4600_60_205, 10 links, 9 joints
Links:
- link base_link: geometry collision mesh filename=package://abb_irb4600_60_205/meshes/collision/base_link.stl; visual mesh filename=package://abb_irb4600_60_205/meshes/visual/base_link.dae
- link link_1: geometry collision mesh filename=package://abb_irb4600_60_205/meshes/collision/link_1.stl; visual mesh filename=package://abb_irb4600_60_205/meshes/visual/link_1.dae
- link link_2: geometry collision mesh filename=package://abb_irb4600_60_205/meshes/collision/link_2.stl; visual mesh filename=package://abb_irb4600_60_205/meshes/visual/link_2.dae
- link link_3: geometry collision mesh filename=package://abb_irb4600_60_205/meshes/collision/link_3.stl; visual mesh filename=package://abb_irb4600_60_205/meshes/visual/link_3.dae
- link link_4: geometry collision mesh filename=package://abb_irb4600_60_205/meshes/collision/link_4.stl; visual mesh filename=package://abb_irb4600_60_205/meshes/visual/link_4.dae
- link link_5: geometry collision mesh filename=package://abb_irb4600_60_205/meshes/collision/link_5.stl; visual mesh filename=package://abb_irb4600_60_205/meshes/visual/link_5.dae
- link link_6: geometry collision mesh filename=package://abb_irb4600_60_205/meshes/collision/link_6.stl; visual mesh filename=package://abb_irb4600_60_205/meshes/visual/link_6.dae

File: urdf/irb4600_60_205_macro.xacro (robot description, xacro)
@@ -11,5 +11,5 @@
       <visual name="visual">
         <geometry>
-          <mesh filename="package://abb_irb4600_60_205/meshes/collision/base_link.stl"/>
+          <mesh filename="package://abb_irb4600_60_205/meshes/visual/base_link.dae"/>
         </geometry>
         <material name="yellow">
@@ -26,5 +26,5 @@
       <visual name="visual">
         <geometry>
-          <mesh filename="package://abb_irb4600_60_205/meshes/collision/link_1.stl"/>
+          <mesh filename="package://abb_irb4600_60_205/meshes/visual/link_1.dae"/>
         </geometry>
         <material name="yellow"/>
@@ -39,5 +39,5 @@
       <visual name="visual">
         <geometry>
-          <mesh filename="package://abb_irb4600_60_205/meshes/collision/link_2.stl"/>
+          <mesh filename="package://abb_irb4600_60_205/meshes/visual/link_2.dae"/>
         </geometry>
         <material name="yellow"/>
@@ -52,5 +52,5 @@
       <visual name="visual">
         <geometry>
-          <mesh filename="package://abb_irb4600_60_205/meshes/collision/link_3.stl"/>
+          <mesh filename="package://abb_irb4600_60_205/meshes/visual/link_3.dae"/>
         </geometry>
         <material name="yellow"/>
@@ -65,5 +65,5 @@
       <visual name="visual">
         <geometry>
-          <mesh filename="package://abb_irb4600_60_205/meshes/collision/link_4.stl"/>
+          <mesh filename="package://abb_irb4600_60_205/meshes/visual/link_4.dae"/>
         </geometry>
         <material name="yellow"/>
@@ -78,5 +78,5 @@
       <visual name="visual">
         <geometry>
-          <mesh filename="package://abb_irb4600_60_205/meshes/collision/link_5.stl"/>
+          <mesh filename="package://abb_irb4600_60_205/meshes/visual/link_5.dae"/>
         </geometry>
         <material name="yellow"/>
@@ -91,5 +91,5 @@
       <visual name="visual">
         <geometry>
-          <mesh filename="package://abb_irb4600_60_205/meshes/collision/link_6.stl"/>
+          <mesh filename="package://abb_irb4600_60_205/meshes/visual/link_6.dae"/>
         </geometry>
         <material name="yellow"/>
